Commit message: Changed into a front wheel drive

File: vehicle/vehicle_model/urdf/actuator.xacro (robot description, xacro)
@@ -25,5 +25,5 @@
   <transmission name="wheel_left_rear_trans">
     <type>transmission_interface/SimpleTransmission</type>
-    <joint name="wheel_left_rear_joint">
+    <joint name="wheel_left_front_joint">
       <hardwareInterface>hardware_interface/VelocityJointInterface</hardwareInterface>
     </joint>
@@ -34,5 +34,5 @@
   <transmission name="wheel_right_rear_trans">
     <type>transmission_interface/SimpleTransmission</type>
-    <joint name="wheel_right_rear_joint">
+    <joint name="wheel_right_front_joint">
       <hardwareInterface>hardware_interface/VelocityJointInterface</hardwareInterface>
     </joint>
