Commit message: Make car move faster

File: vehicle/vehicle_model/urdf/wheel.xacro (robot description, xacro)
@@ -3,5 +3,5 @@
   <xacro:macro name="wheel_macro" params="suffix parent x y yaw radius width">
     <xacro:property name="pi" value="3.1415926835897931" />
-    <xacro:property name="mass" value="40" />
+    <xacro:property name="mass" value="0.5" />
     <joint name="${suffix}_joint" type="continuous">
       <origin rpy="0 0 ${pi/2}" xyz="${x} ${y} 0"/>

Commit message: Fix vehicle params

File: vehicle/vehicle_model/urdf/wheel.xacro (robot description, xacro)
@@ -3,5 +3,5 @@
   <xacro:macro name="wheel_macro" params="suffix parent x y yaw radius width">
     <xacro:property name="pi" value="3.1415926835897931" />
-    <xacro:property name="mass" value="0.5" />
+    <xacro:property name="mass" value="0.05" />
     <joint name="${suffix}_joint" type="continuous">
       <origin rpy="0 0 ${pi/2}" xyz="${x} ${y} 0"/>
@@ -11,5 +11,5 @@
       <dynamics damping="0.1"/>
       <limit effort="50000" velocity="50" />
-      <joint_properties damping="0.0" friction="0.0" />
+      <joint_properties damping="0.001" friction="0.001" />
     </joint>
     <link name="${suffix}_link">
@@ -19,7 +19,4 @@
         </geometry>
         <origin xyz="0 0 0" rpy="0 0 ${yaw}"/>
-        <material name="gray">
-          <color rgba="${25/255} ${25/255} ${25/255} .5"/>
-        </material>
       </visual>
       <inertial>
@@ -33,4 +30,9 @@
           <cylinder radius="${radius}" length="${width}" />
         </geometry>
+        <surface>
+          <friction><!-- Assume very sticky tire (max friction coeff) -->
+            <ode><mu>1.0</mu><mu2>1.0</mu2></ode>
+          </friction>
+        </surface>
       </collision>
     </link>
