Commit message: Gyumin changed car model

File: vehicle/vehicle_model/urdf/body.xacro (robot description, xacro)
@@ -22,7 +22,7 @@
         </geometry> -->
         <!-- <origin xyz="${wheel_base/2} 0 ${vehicle_height/2}" rpy="0 ${-pi/2} ${pi/2}"/> -->
-        <origin xyz="0 0 0" rpy="0 0 0"/>
+        <origin xyz="0.025 -0.01 -0.085" rpy="1.570796 0 1.5707963"/>
         <geometry>
-          <mesh filename="package://vehicle_model/mesh/body.dae" scale="${wheel_base/2.85} 1 1"/>
+          <mesh filename="package://vehicle_model/mesh/car4.dae" scale="1 1 1"/>
         </geometry>
         <material name="black">

File: vehicle/vehicle_model/urdf/steering.xacro (robot description, xacro)
@@ -3,5 +3,5 @@
   <xacro:macro name="steering_macro" params="suffix parent x y yaw length">
     <xacro:property name="pi" value="3.1415926835897931" />
-    <xacro:property name="radius" value="0.1" />
+    <xacro:property name="radius" value="0.01" />
     <xacro:property name="length" value="0.01" />
     <xacro:property name="mass" value="10.0" />
@@ -40,5 +40,5 @@
   <xacro:macro name="steering_link_macro" params="suffix parent x y">
     <xacro:property name="pi" value="3.1415926835897931" />
-    <xacro:property name="radius" value="0.1" />
+    <xacro:property name="radius" value="0.01" />
     <xacro:property name="length" value="0.01" />
     <xacro:property name="mass" value="10.0" />

File: vehicle/vehicle_model/urdf/vehicle.xacro (robot description, xacro)
@@ -35,11 +35,11 @@
   <!-- steering-->
   <xacro:steering_link_macro suffix="steering_front" parent="base_link" x="${wheel_base}" y="0"/>
-  <xacro:steering_macro suffix="steering_right_front" parent="steering_front_link" x="0" y="${-1*wheel_tread/2}" yaw="0" length="${wheel_width}"/>
-  <xacro:steering_macro suffix="steering_left_front" parent="steering_front_link" x="0" y="${wheel_tread/2}" yaw="0" length="${wheel_width}"/>
+  <xacro:steering_macro suffix="steering_right_front" parent="steering_front_link" x="0" y="${-1*wheel_tread}" yaw="0" length="${wheel_width}"/>
+  <xacro:steering_macro suffix="steering_left_front" parent="steering_front_link" x="0" y="${wheel_tread}" yaw="0" length="${wheel_width}"/>
   <!-- wheel -->
   <xacro:wheel_macro suffix="wheel_right_front" parent="steering_right_front_link" x="0" y="0" yaw="${pi}" radius="${wheel_radius}" width="${wheel_width}"/>
   <xacro:wheel_macro suffix="wheel_left_front" parent="steering_left_front_link" x="0" y="0" yaw="0" radius="${wheel_radius}" width="${wheel_width}"/>
-  <xacro:wheel_macro suffix="wheel_right_rear" parent="base_link" x="0" y="${-1*wheel_tread/2}" yaw="${pi}" radius="${wheel_radius}" width="${wheel_width}"/>
-  <xacro:wheel_macro suffix="wheel_left_rear" parent="base_link" x="0" y="${wheel_tread/2}" yaw="0" radius="${wheel_radius}" width="${wheel_width}"/>
+  <xacro:wheel_macro suffix="wheel_right_rear" parent="base_link" x="0" y="${-1*wheel_tread/1.6}" yaw="${pi}" radius="${wheel_radius}" width="${wheel_width}"/>
+  <xacro:wheel_macro suffix="wheel_left_rear" parent="base_link" x="0" y="${wheel_tread/1.6}" yaw="0" radius="${wheel_radius}" width="${wheel_width}"/>
   <!-- actuator -->
  	<xacro:include filename="$(find vehicle_model)/urdf/actuator.xacro"/>

File: vehicle/vehicle_model/urdf/wheel.xacro (robot description, xacro)
@@ -16,5 +16,5 @@
       <visual>
         <geometry>
-          <mesh filename="package://vehicle_model/mesh/wheel.dae" scale="${3*radius} ${3*radius} ${3*radius}"/>
+          <mesh filename="package://vehicle_model/mesh/wheel.dae" scale="0.12 0.12 0.12"/>
         </geometry>
         <origin xyz="0 0 0" rpy="0 0 ${yaw}"/>

Commit message: Fix hcpath action message generation

File: vehicle/vehicle_model/urdf/body.xacro (robot description, xacro)
@@ -17,9 +17,4 @@
       </inertial>
       <visual>
-        <!-- <origin xyz="${wheel_base/2} 0 ${vehicle_height/2}" rpy="0 0 0"/>
-        <geometry>
-          <box size="${vehicle_length} 0.9 ${vehicle_height}"/>
-        </geometry> -->
-        <!-- <origin xyz="${wheel_base/2} 0 ${vehicle_height/2}" rpy="0 ${-pi/2} ${pi/2}"/> -->
         <origin xyz="0.025 -0.01 -0.085" rpy="1.570796 0 1.5707963"/>
         <geometry>

File: vehicle/vehicle_model/urdf/wheel.xacro (robot description, xacro)
@@ -23,5 +23,7 @@
         <origin xyz="0 0 0" rpy="0 0 0"/>
         <mass value="${mass}"/>
-        <inertia ixx="${mass*radius*radius/2}"  ixy="0"  ixz="0" iyy="${radius*radius*mass/4+width*width*mass/12}" iyz="0" izz="${radius*radius*mass/4+width*width*mass/12}" />
+        <inertia ixx="${mass*radius*radius/2}"  ixy="0"  ixz="0"
+          iyy="${radius*radius*mass/4+width*width*mass/12}" iyz="0"
+            izz="${radius*radius*mass/4+width*width*mass/12}" />
       </inertial>
       <collision>

Commit message: Changed vehicle info, and wheel scale size

File: vehicle/vehicle_model/urdf/body.xacro (robot description, xacro)
@@ -28,5 +28,5 @@
         <origin xyz="${wheel_base/2} 0 ${vehicle_height/2}" rpy="0 0 0"/>
         <geometry>
-          <box size="${vehicle_length} 0.9 ${vehicle_height}"/>
+          <box size="${vehicle_length} ${vehicle_width} ${vehicle_height}"/>
         </geometry>
       </collision>

File: vehicle/vehicle_model/urdf/wheel.xacro (robot description, xacro)
@@ -16,5 +16,5 @@
       <visual>
         <geometry>
-          <mesh filename="package://vehicle_model/mesh/wheel.dae" scale="0.12 0.12 0.12"/>
+          <mesh filename="package://vehicle_model/mesh/wheel.dae" scale="0.15 0.15 0.15"/>
         </geometry>
         <origin xyz="0 0 0" rpy="0 0 ${yaw}"/>

Commit message: Added truck with fifth wheel and side hitch

File: vehicle/vehicle_model/urdf/body.xacro (robot description, xacro)
@@ -19,5 +19,5 @@
         <origin xyz="0.025 -0.01 -0.085" rpy="1.570796 0 1.5707963"/>
         <geometry>
-          <mesh filename="package://vehicle_model/mesh/car4.dae" scale="1 1 1"/>
+          <mesh filename="package://vehicle_model/mesh/car_fifthwheel.dae" scale="1 1 1"/>
         </geometry>
         <material name="black">

Commit message: Add contact sensors on the kingpin and the side hitches

File: vehicle/vehicle_model/urdf/body.xacro (robot description, xacro)
@@ -19,5 +19,5 @@
         <origin xyz="0.025 -0.01 -0.085" rpy="1.570796 0 1.5707963"/>
         <geometry>
-          <mesh filename="package://vehicle_model/mesh/car_fifthwheel.dae" scale="1 1 1"/>
+          <mesh filename="package://vehicle_model/mesh/car_sidehitch.dae" scale="1 1 1"/>
         </geometry>
         <material name="black">

Commit message: Added V-shaped collision material, and contact sensor

File: vehicle/vehicle_model/urdf/body.xacro (robot description, xacro)
@@ -19,5 +19,5 @@
         <origin xyz="0.025 -0.01 -0.085" rpy="1.570796 0 1.5707963"/>
         <geometry>
-          <mesh filename="package://vehicle_model/mesh/car_sidehitch.dae" scale="1 1 1"/>
+          <mesh filename="package://vehicle_model/mesh/car_fifthwheel.dae" scale="1 1 1"/>
         </geometry>
         <material name="black">
@@ -29,4 +29,103 @@
         <geometry>
           <box size="${vehicle_length} ${vehicle_width} ${vehicle_height}"/>
+        </geometry>
+      </collision>
+    </link>
+    <joint name="${suffix}_kingpin_joint1" type="fixed">
+      <parent link="${parent}"/>
+      <origin rpy="0 0 0" xyz="0 0 0"/>
+      <child  link="${suffix}_kingpin1"/>
+    </joint>
+    <link name="${suffix}_kingpin1">
+      <inertial>
+        <origin xyz="0 0 0" rpy="0 0 0"/>
+        <mass value="0.01"/>
+        <inertia ixx="0.1" ixy="0.0" ixz="0.0"
+                 iyy="0.1" iyz="0.0"
+                 izz="0.1"/>
+      </inertial>
+      <visual>
+        <origin xyz="0.125 0 0.145" rpy="0 0 0"/>
+        <geometry>
+          <box size="0.024 0.024 0.024"/>
+        </geometry>
+        <material name="black">
+            <color rgba="${25/255} ${25/255} ${25/255} .9"/>
+        </material>
+      </visual>
+      <collision name="kingpin_collision">
+        <origin xyz="0.125 0 0.145" rpy="0 0 0"/>
+        <geometry>
+          <box size="0.024 0.024 0.024"/>
+        </geometry>
+      </collision>
+    <sensor name='kingpin_sensor' type='contact'>
+        <always_on>1</always_on>
+        <contact>
+          <collision>kingpin_collision</collision>
+          <topic>__default_topic__</topic>
+        </contact>
+        <plugin name='contact_sensor_plugin' filename='libgazebo_ros_bumper.so'>
+          <bumperTopicName>kingpin_contact</bumperTopicName>
+          <frameName>kingpin</frameName>
+        </plugin>
+        <pose frame=''>0 0 0.4075 0 -0 0</pose>
+      </sensor>
+    </link>
+    <joint name="${suffix}_kingpin_joint2" type="fixed">
+      <parent link="${parent}"/>
+      <origin rpy="0 0 0" xyz="0 0 0"/>
+      <child  link="${suffix}_kingpin2"/>
+    </joint>
+    <link name="${suffix}_kingpin2">
+      <inertial>
+        <origin xyz="0 0 0" rpy="0 0 0"/>
+        <mass value="0.01"/>
+        <inertia ixx="0.1" ixy="0.0" ixz="0.0"
+                 iyy="0.1" iyz="0.0"
+                 izz="0.1"/>
+      </inertial>
+      <visual>
+        <origin xyz="0.09 -0.022 0.145" rpy="0 0 0.2617994"/>
+        <geometry>
+          <box size="0.05 0.01 0.024"/>
+        </geometry>
+        <material name="black">
+            <color rgba="${25/255} ${25/255} ${25/255} .9"/>
+        </material>
+      </visual>
+      <collision>
+        <origin xyz="0.09 -0.022 0.145" rpy="0 0 0.2617994"/>
+        <geometry>
+          <box size="0.05 0.01 0.024"/>
+        </geometry>
+      </collision>
+    </link>
+    <joint name="${suffix}_kingpin_joint3" type="fixed">
+      <parent link="${parent}"/>
+      <origin rpy="0 0 0" xyz="0 0 0"/>
+      <child  link="${suffix}_kingpin3"/>
+    </joint>
+    <link name="${suffix}_kingpin3">
+      <inertial>
+        <origin xyz="0 0 0" rpy="0 0 0"/>
+        <mass value="0.01"/>
+        <inertia ixx="0.1" ixy="0.0" ixz="0.0"
+                 iyy="0.1" iyz="0.0"
+                 izz="0.1"/>
+      </inertial>
+      <visual>
+        <origin xyz="0.09 0.022 0.145" rpy="0 0 -0.2617994"/>
+        <geometry>
+          <box size="0.05 0.01 0.024"/>
+        </geometry>
+        <material name="black">
+            <color rgba="${25/255} ${25/255} ${25/255} .9"/>
+        </material>
+      </visual>
+      <collision>
+        <origin xyz="0.09 0.022 0.145" rpy="0 0 -0.2617994"/>
+        <geometry>
+          <box size="0.05 0.01 0.024"/>
         </geometry>
       </collision>

Commit message: Added L,R fender and skirt

File: vehicle/vehicle_model/urdf/body.xacro (robot description, xacro)
@@ -131,4 +131,132 @@
       </collision>
     </link>
+    <joint name="${suffix}_L_fender_joint" type="fixed">
+      <parent link="${parent}"/>
+      <origin rpy="0 0 0" xyz="0 0 0"/>
+      <child  link="${suffix}_L_fender"/>
+    </joint>
+    <link name="${suffix}_L_fender">
+      <inertial>
+        <origin xyz="0 0 0" rpy="0 0 0"/>
+        <mass value="0.01"/>
+        <inertia ixx="0.1" ixy="0.0" ixz="0.0"
+                 iyy="0.1" iyz="0.0"
+                 izz="0.1"/>
+      </inertial>
+      <visual>
+        <origin xyz="-0.06 0.1 0.08" rpy="1.5707963 0 0"/>
+        <geometry>
+          <cylinder radius="0.005" length="0.15"/>
+        </geometry>
+        <material name="black">
+            <color rgba="${25/255} ${25/255} ${25/255} .9"/>
+        </material>
+      </visual>
+      <collision name="L_fender_collision">
+        <origin xyz="-0.06 0.1 0.08" rpy="1.5707963 0 0"/>
+        <geometry>
+           <cylinder radius="0.005" length="0.15"/>
+        </geometry>
+      </collision>
+    <sensor name='L_fender_sensor' type='contact'>
+        <always_on>1</always_on>
+        <contact>
+          <collision>L_fender_collision</collision>
+          <topic>__default_topic__</topic>
+        </contact>
+        <plugin name='L_fender_contact_sensor_plugin' filename='libgazebo_ros_bumper.so'>
+          <bumperTopicName>L_fender_contact</bumperTopicName>
+          <frameName>L_fender</frameName>
+        </plugin>
+        <pose frame=''>0 0 0.4075 0 -0 0</pose>
+      </sensor>
+    </link>
+<joint name="${suffix}_L_skirt_joint" type="fixed">
+      <parent link="${parent}"/>
+      <origin rpy="0 0 0" xyz="0 0 0"/>
+      <child  link="${suffix}_L_skirt"/>
+    </joint>
+    <link name="${suffix}_L_skirt">
+      <inertial>
+        <origin xyz="0 0 0" rpy="0 0 0"/>
+        <mass value="0.01"/>
+        <inertia ixx="0.1" ixy="0.0" ixz="0.0"
+                 iyy="0.1" iyz="0.0"
+                 izz="0.1"/>
+      </inertial>
+      <visual>
+        <origin xyz="-0.06 0.145 0.045" rpy="0 0 0"/>
+        <geometry>
+          <box size="0.001 0.06 0.06"/>
+        </geometry>
+        <material name="black">
+            <color rgba="${25/255} ${25/255} ${25/255} .9"/>
+        </material>
+      </visual>
+    </link>
+    <joint name="${suffix}_R_fender_joint" type="fixed">
+      <parent link="${parent}"/>
+      <origin rpy="0 0 0" xyz="0 0 0"/>
+      <child  link="${suffix}_R_fender"/>
+    </joint>
+    <link name="${suffix}_R_fender">
+      <inertial>
+        <origin xyz="0 0 0" rpy="0 0 0"/>
+        <mass value="0.01"/>
+        <inertia ixx="0.1" ixy="0.0" ixz="0.0"
+                 iyy="0.1" iyz="0.0"
+                 izz="0.1"/>
+      </inertial>
+      <visual>
+        <origin xyz="-0.06 -0.1 0.08" rpy="1.5707963 0 0"/>
+        <geometry>
+          <cylinder radius="0.005" length="0.15"/>
+        </geometry>
+        <material name="black">
+            <color rgba="${25/255} ${25/255} ${25/255} .9"/>
+        </material>
+      </visual>
+      <collision name="R_fender_collision">
+        <origin xyz="-0.06 -0.1 0.08" rpy="1.5707963 0 0"/>
+        <geometry>
+           <cylinder radius="0.005" length="0.15"/>
+        </geometry>
+      </collision>
+    <sensor name='R_fender_sensor' type='contact'>
+        <always_on>1</always_on>
+        <contact>
+          <collision>R_fender_collision</collision>
+          <topic>__default_topic__</topic>
+        </contact>
+        <plugin name='R_fender_contact_sensor_plugin' filename='libgazebo_ros_bumper.so'>
+          <bumperTopicName>R_fender_contact</bumperTopicName>
+          <frameName>R_fender</frameName>
+        </plugin>
+        <pose frame=''>0 0 0.4075 0 -0 0</pose>
+      </sensor>
+    </link>
+<joint name="${suffix}_R_skirt_joint" type="fixed">
+      <parent link="${parent}"/>
+      <origin rpy="0 0 0" xyz="0 0 0"/>
+      <child  link="${suffix}_R_skirt"/>
+    </joint>
+    <link name="${suffix}_R_skirt">
+      <inertial>
+        <origin xyz="0 0 0" rpy="0 0 0"/>
+        <mass value="0.01"/>
+        <inertia ixx="0.1" ixy="0.0" ixz="0.0"
+                 iyy="0.1" iyz="0.0"
+                 izz="0.1"/>
+      </inertial>
+      <visual>
+        <origin xyz="-0.06 -0.145 0.045" rpy="0 0 0"/>
+        <geometry>
+          <box size="0.001 0.06 0.06"/>
+        </geometry>
+        <material name="black">
+            <color rgba="${25/255} ${25/255} ${25/255} .9"/>
+        </material>
+      </visual>
+   </link>
     <light name='under' type='directional'>
       <cast_shadows>1</cast_shadows>

Commit message: bottom markers + GMC's collision elements

File: vehicle/vehicle_model/urdf/body.xacro (robot description, xacro)
@@ -32,16 +32,16 @@
       </collision>
     </link>
-    <joint name="${suffix}_kingpin_joint1" type="fixed">
-      <parent link="${parent}"/>
-      <origin rpy="0 0 0" xyz="0 0 0"/>
-      <child  link="${suffix}_kingpin1"/>
-    </joint>
-    <link name="${suffix}_kingpin1">
-      <inertial>
-        <origin xyz="0 0 0" rpy="0 0 0"/>
-        <mass value="0.01"/>
-        <inertia ixx="0.1" ixy="0.0" ixz="0.0"
-                 iyy="0.1" iyz="0.0"
-                 izz="0.1"/>
+    <joint name="${suffix}_5whl_joint1" type="fixed">
+      <parent link="${parent}"/>
+      <origin rpy="0 0 0" xyz="0 0 0"/>
+      <child  link="${suffix}_5whl1"/>
+    </joint>
+    <link name="${suffix}_5whl1">
+      <inertial>
+        <origin xyz="0 0 0" rpy="0 0 0"/>
+        <mass value="0.01"/>
+        <inertia ixx="0.001" ixy="0.0" ixz="0.0"
+                 iyy="0.001" iyz="0.0"
+                 izz="0.001"/>
       </inertial>
       <visual>
@@ -54,5 +54,5 @@
         </material>
       </visual>
-      <collision name="kingpin_collision">
+      <collision name="5whl_collision">
         <origin xyz="0.125 0 0.145" rpy="0 0 0"/>
         <geometry>
@@ -60,29 +60,29 @@
         </geometry>
       </collision>
-    <sensor name='kingpin_sensor' type='contact'>
+    <sensor name='5whl_sensor' type='contact'>
         <always_on>1</always_on>
         <contact>
-          <collision>kingpin_collision</collision>
+          <collision>5whl_collision</collision>
           <topic>__default_topic__</topic>
         </contact>
         <plugin name='contact_sensor_plugin' filename='libgazebo_ros_bumper.so'>
-          <bumperTopicName>kingpin_contact</bumperTopicName>
-          <frameName>kingpin</frameName>
+          <bumperTopicName>5whl_contact</bumperTopicName>
+          <frameName>5whl</frameName>
         </plugin>
         <pose frame=''>0 0 0.4075 0 -0 0</pose>
       </sensor>
     </link>
-    <joint name="${suffix}_kingpin_joint2" type="fixed">
-      <parent link="${parent}"/>
-      <origin rpy="0 0 0" xyz="0 0 0"/>
-      <child  link="${suffix}_kingpin2"/>
-    </joint>
-    <link name="${suffix}_kingpin2">
-      <inertial>
-        <origin xyz="0 0 0" rpy="0 0 0"/>
-        <mass value="0.01"/>
-        <inertia ixx="0.1" ixy="0.0" ixz="0.0"
-                 iyy="0.1" iyz="0.0"
-                 izz="0.1"/>
+    <joint name="${suffix}_5whl_joint2" type="fixed">
+      <parent link="${parent}"/>
+      <origin rpy="0 0 0" xyz="0 0 0"/>
+      <child  link="${suffix}_5whl2"/>
+    </joint>
+    <link name="${suffix}_5whl2">
+      <inertial>
+        <origin xyz="0 0 0" rpy="0 0 0"/>
+        <mass value="0.01"/>
+        <inertia ixx="0.001" ixy="0.0" ixz="0.0"
+                 iyy="0.001" iyz="0.0"
+                 izz="0.001"/>
       </inertial>
       <visual>
@@ -102,16 +102,16 @@
       </collision>
     </link>
-    <joint name="${suffix}_kingpin_joint3" type="fixed">
-      <parent link="${parent}"/>
-      <origin rpy="0 0 0" xyz="0 0 0"/>
-      <child  link="${suffix}_kingpin3"/>
-    </joint>
-    <link name="${suffix}_kingpin3">
-      <inertial>
-        <origin xyz="0 0 0" rpy="0 0 0"/>
-        <mass value="0.01"/>
-        <inertia ixx="0.1" ixy="0.0" ixz="0.0"
-                 iyy="0.1" iyz="0.0"
-                 izz="0.1"/>
+    <joint name="${suffix}_5whl_joint3" type="fixed">
+      <parent link="${parent}"/>
+      <origin rpy="0 0 0" xyz="0 0 0"/>
+      <child  link="${suffix}_5whl3"/>
+    </joint>
+    <link name="${suffix}_5whl3">
+      <inertial>
+        <origin xyz="0 0 0" rpy="0 0 0"/>
+        <mass value="0.01"/>
+        <inertia ixx="0.001" ixy="0.0" ixz="0.0"
+                 iyy="0.001" iyz="0.0"
+                 izz="0.001"/>
       </inertial>
       <visual>
@@ -140,7 +140,7 @@
         <origin xyz="0 0 0" rpy="0 0 0"/>
         <mass value="0.01"/>
-        <inertia ixx="0.1" ixy="0.0" ixz="0.0"
-                 iyy="0.1" iyz="0.0"
-                 izz="0.1"/>
+        <inertia ixx="0.01" ixy="0.0" ixz="0.0"
+                 iyy="0.01" iyz="0.0"
+                 izz="0.01"/>
       </inertial>
       <visual>
@@ -159,5 +159,5 @@
         </geometry>
       </collision>
-    <sensor name='L_fender_sensor' type='contact'>
+      <sensor name='L_fender_sensor' type='contact'>
         <always_on>1</always_on>
         <contact>
@@ -172,5 +172,5 @@
       </sensor>
     </link>
-<joint name="${suffix}_L_skirt_joint" type="fixed">
+    <joint name="${suffix}_L_skirt_joint" type="fixed">
       <parent link="${parent}"/>
       <origin rpy="0 0 0" xyz="0 0 0"/>
@@ -181,7 +181,7 @@
         <origin xyz="0 0 0" rpy="0 0 0"/>
         <mass value="0.01"/>
-        <inertia ixx="0.1" ixy="0.0" ixz="0.0"
-                 iyy="0.1" iyz="0.0"
-                 izz="0.1"/>
+        <inertia ixx="0.01" ixy="0.0" ixz="0.0"
+                 iyy="0.01" iyz="0.0"
+                 izz="0.01"/>
       </inertial>
       <visual>
@@ -204,7 +204,7 @@
         <origin xyz="0 0 0" rpy="0 0 0"/>
         <mass value="0.01"/>
-        <inertia ixx="0.1" ixy="0.0" ixz="0.0"
-                 iyy="0.1" iyz="0.0"
-                 izz="0.1"/>
+        <inertia ixx="0.01" ixy="0.0" ixz="0.0"
+                 iyy="0.01" iyz="0.0"
+                 izz="0.01"/>
       </inertial>
       <visual>
@@ -223,5 +223,5 @@
         </geometry>
       </collision>
-    <sensor name='R_fender_sensor' type='contact'>
+      <sensor name='R_fender_sensor' type='contact'>
         <always_on>1</always_on>
         <contact>
@@ -236,5 +236,5 @@
       </sensor>
     </link>
-<joint name="${suffix}_R_skirt_joint" type="fixed">
+    <joint name="${suffix}_R_skirt_joint" type="fixed">
       <parent link="${parent}"/>
       <origin rpy="0 0 0" xyz="0 0 0"/>
@@ -245,7 +245,7 @@
         <origin xyz="0 0 0" rpy="0 0 0"/>
         <mass value="0.01"/>
-        <inertia ixx="0.1" ixy="0.0" ixz="0.0"
-                 iyy="0.1" iyz="0.0"
-                 izz="0.1"/>
+        <inertia ixx="0.01" ixy="0.0" ixz="0.0"
+                 iyy="0.01" iyz="0.0"
+                 izz="0.01"/>
       </inertial>
       <visual>

File: vehicle/vehicle_model/urdf/vehicle.xacro (robot description, xacro)
@@ -48,5 +48,5 @@
   <!-- ================ sensor to base_link xforms ================ -->
 	<xacro:property name="calibration" value="${load_yaml('$(find vehicle_model)/config/calibration.yaml')}"/>
-  <xacro:quad_camera_macro parent="base_link"
+  <!-- xacro:quad_camera_macro parent="base_link"
       x="${calibration['base_link2quad']['x']}"
       y="${calibration['base_link2quad']['y']}"
@@ -55,5 +55,5 @@
       pitch="${calibration['base_link2quad']['pitch']}"
       yaw="${calibration['base_link2quad']['yaw']}"
-      fps="6" width="1280" height="720" fov="1.6"/>
+      fps="6" width="1280" height="720" fov="1.6"/-->
   <xacro:monocular_camera_macro prefix="webcam" parent="base_link"
       x="${calibration['base_link2camera']['x']}"
