Commit message: Rear trucks successfully contacts the kingpin!

File: vehicle/vehicle_model/urdf/rear_body.xacro (robot description, xacro)
@@ -19,5 +19,5 @@
         <origin xyz="0.025 -0.01 -0.085" rpy="1.570796 0 1.5707963"/>
         <geometry>
-          <mesh filename="package://vehicle_model/mesh/car_sidehitch_5whl.dae" scale="1 1 1"/>
+          <mesh filename="package://vehicle_model/mesh/car_no_cam.dae" scale="1 1 1"/>
         </geometry>
         <material name="black">
