Commit message: gazebo_empty_world.launch works

File: vehicle/sensor_model/camera/camera_description/urdf/monocular_camera.xacro (robot description, xacro)
@@ -17,5 +17,5 @@
         <origin rpy="0 0 0" xyz="0 0 0"/>
         <material name="red">
-          <color rgba="1.0 0.0 0.0 2.0"/>
+          <color rgba="${255/255} ${108/255} ${10/255} 1.0"/>
         </material>
       </visual>

File: vehicle/sensor_model/imu/imu_description/urdf/imu.xacro (robot description, xacro)
@@ -17,5 +17,5 @@
         <origin rpy="0 0 0" xyz="0 0 0"/>
         <material name="red">
-          <color rgba="1.0 0.0 0.0 2.0"/>
+          <color rgba="${255/255} ${108/255} ${10/255} 1.0"/>
         </material>
       </visual>

File: vehicle/vehicle_model/urdf/body.xacro (robot description, xacro)
@@ -27,5 +27,5 @@
         </geometry>
         <material name="black">
-            <color rgba="0.1 0.1 0.1 0.5"/>
+            <color rgba="${25/255} ${25/255} ${25/255} .9"/>
         </material>
       </visual>

File: vehicle/vehicle_model/urdf/steering.xacro (robot description, xacro)
@@ -20,5 +20,5 @@
         <origin xyz="0 0 0" rpy="${pi/2} 0 0"/>
         <material name="black">
-          <color rgba="0.1 0.1 0.1 2.0"/>
+          <color rgba="${25/255} ${25/255} ${25/255} 0.9"/>
         </material>
       </visual>
@@ -55,5 +55,5 @@
         <origin xyz="0 0 0" rpy="${pi/2} 0 0"/>
         <material name="black">
-          <color rgba="0.1 0.1 0.1 2.0"/>
+          <color rgba="${25/255} ${25/255} ${25/255} 0.9"/>
         </material>
       </visual>

File: vehicle/vehicle_model/urdf/vehicle.xacro (robot description, xacro)
@@ -4,6 +4,4 @@
   <xacro:include filename="$(find vehicle_model)/urdf/wheel.xacro" />
   <xacro:include filename="$(find vehicle_model)/urdf/steering.xacro" />
-  <xacro:include filename="$(find velodyne_description)/urdf/HDL-32E.urdf.xacro"/>
-  <xacro:include filename="$(find velodyne_description)/urdf/VLP-16.urdf.xacro"/>
   <xacro:include filename="$(find camera_description)/urdf/monocular_camera.xacro"/>
   <xacro:include filename="$(find imu_description)/urdf/imu.xacro"/>
@@ -49,8 +47,4 @@
   <!-- ================ sensor ================ -->
 	<xacro:property name="calibration" value="${load_yaml('$(find vehicle_model)/config/calibration.yaml')}"/>
-  <HDL-32E parent="base_link" name="velodyne" topic="/points_raw" hz="10" samples="220" gpu="$(arg gpu)">
-    <origin xyz="${calibration['base_link2velodyne']['x']} ${calibration['base_link2velodyne']['y']} ${calibration['base_link2velodyne']['z']}"
-            rpy="${calibration['base_link2velodyne']['roll']} ${calibration['base_link2velodyne']['pitch']} ${calibration['base_link2velodyne']['yaw']}" />
-  </HDL-32E>
   <xacro:monocular_camera_macro suffix="camera" parent="base_link" namespace=""
                                 x="${calibration['base_link2camera']['x']}"

File: vehicle/vehicle_model/urdf/wheel.xacro (robot description, xacro)
@@ -20,5 +20,5 @@
         <origin xyz="0 0 0" rpy="0 0 ${yaw}"/>
         <material name="gray">
-          <color rgba="0.1 0.1 0.1 2.0"/>
+          <color rgba="${25/255} ${25/255} ${25/255} .5"/>
         </material>
       </visual>

Commit message: Fix rear wheels not getting TF'ed

File: vehicle/sensor_model/camera/camera_description/urdf/monocular_camera.xacro (robot description, xacro)
@@ -4,6 +4,6 @@
   <xacro:macro name="monocular_camera_macro"
     params="prefix parent x y z roll pitch yaw fps width height fov">
-    <xacro:property name="len" value="0.2" />
-    <xacro:property name="mass" value="0.1" />
+    <xacro:property name="len" value="0.001" />
+    <xacro:property name="mass" value="0.010" />
     <joint name="${prefix}_joint" type="fixed">
       <origin rpy="${roll} ${pitch} ${yaw}" xyz="${x} ${y} ${z}"/>
@@ -13,12 +13,8 @@
     <link name="${prefix}_link">
       <visual>
-        <geometry><cylinder length="${len}" radius="0.02"/></geometry>
-        <origin rpy="0 0 0" xyz="0 0 0"/>
-        <material name="red">
-          <color rgba="${255/255} ${108/255} ${10/255} 1.0"/>
-        </material>
+        <geometry><box size="${len} ${len} ${len}"/></geometry>
+        <material name="black"><color rgba="0 0 0 1.0"/></material>
       </visual>
       <inertial>
-        <origin rpy="0 0 0" xyz="0 0 0"/>
         <mass value="${mass}"/>
         <inertia ixx="${(len*len+len*len)*mass/12.0}" ixy="0.0" ixz="0.0"
@@ -27,6 +23,5 @@
       </inertial>
       <collision>
-        <origin rpy="0 0 0" xyz="0 0 0"/>
-        <geometry><cylinder length="${len}" radius="0.02"/></geometry>
+        <geometry><box size="${len} ${len} ${len}"/></geometry>
       </collision>
     </link>

File: vehicle/vehicle_model/urdf/actuator.xacro (robot description, xacro)
@@ -22,20 +22,20 @@
     </actuator>
   </transmission>
-  <!-- rear wheel motor -->
-  <transmission name="wheel_left_rear_trans">
+  <!-- front wheel motor -->
+  <transmission name="wheel_left_front_trans">
     <type>transmission_interface/SimpleTransmission</type>
     <joint name="wheel_left_front_joint">
       <hardwareInterface>hardware_interface/VelocityJointInterface</hardwareInterface>
     </joint>
-    <actuator name="wheel_left_rear_motor">
+    <actuator name="wheel_left_front_motor">
        <mechanismReduction>1</mechanismReduction>
     </actuator>
   </transmission>
-  <transmission name="wheel_right_rear_trans">
+  <transmission name="wheel_right_front_trans">
     <type>transmission_interface/SimpleTransmission</type>
     <joint name="wheel_right_front_joint">
       <hardwareInterface>hardware_interface/VelocityJointInterface</hardwareInterface>
     </joint>
-    <actuator name="wheel_right_rear_motor">
+    <actuator name="wheel_right_front_motor">
        <mechanismReduction>1</mechanismReduction>
     </actuator>

File: vehicle/vehicle_model/urdf/steering.xacro (robot description, xacro)
@@ -5,5 +5,5 @@
     <xacro:property name="radius" value="0.01" />
     <xacro:property name="length" value="0.01" />
-    <xacro:property name="mass" value="10.0" />
+    <xacro:property name="mass" value="1" />
     <joint name="${suffix}_joint" type="revolute">
       <origin rpy="0 0 0" xyz="${x} ${y} 0"/>
@@ -11,5 +11,5 @@
       <child  link="${suffix}_link"/>
       <axis xyz="0 0 1"/>
-      <limit effort="100000000.0" lower="-0.6" upper="0.6" velocity="0.5"/>
+      <limit effort="100000000.0" lower="-0.6" upper="0.6" velocity="1"/>
     </joint>
     <link name="${suffix}_link">
@@ -42,5 +42,5 @@
     <xacro:property name="radius" value="0.01" />
     <xacro:property name="length" value="0.01" />
-    <xacro:property name="mass" value="10.0" />
+    <xacro:property name="mass" value="0.3" />
     <joint name="${suffix}_joint" type="fixed">
       <origin rpy="0 0 0" xyz="${x} ${y} 0"/>

Commit message: Shrink the bottom marker size, to fit 16x12 markers

File: vehicle/sensor_model/camera/camera_description/urdf/monocular_camera.xacro (robot description, xacro)
@@ -4,6 +4,6 @@
   <xacro:macro name="monocular_camera_macro"
     params="prefix parent x y z roll pitch yaw fps width height fov">
-    <xacro:property name="len" value="0.001" />
-    <xacro:property name="mass" value="0.010" />
+    <xacro:property name="len" value="0.01" />
+    <xacro:property name="mass" value="0.050" />
     <joint name="${prefix}_joint" type="fixed">
       <origin rpy="${roll} ${pitch} ${yaw}" xyz="${x} ${y} ${z}"/>
