Commit message: ArucoNode works with quad camera

File: vehicle/sensor_model/camera/camera_description/urdf/D430IR.xacro (robot description, xacro)
@@ -1,18 +1,15 @@
 <?xml version="1.0"?>
 <robot xmlns:xacro="http://ros.org/wiki/xacro">
-  <xacro:property name="pi" value="3.1415926835897931" />
-  <xacro:macro name="monocular_camera_macro"
-    params="prefix parent x y z roll pitch yaw fps width height fov">
-    <xacro:property name="len" value="0.2" />
-    <xacro:property name="mass" value="0.1" />
-    <joint name="${prefix}_joint" type="fixed">
-      <origin rpy="${roll} ${pitch} ${yaw}" xyz="${x} ${y} ${z}"/>
-      <parent link="${parent}"/>
-      <child  link="${prefix}_link"/>
+  <!-- xacro:property name="pi" value="3.1415926835897931" /-->
+  <xacro:macro name="D430IR_macro"
+    params="parent instance yaw x y z fps width height fov">
+    <joint name="quad${instance}_joint" type="fixed">
+      <origin rpy="0 0 ${yaw}" xyz="${x} ${y} ${z}"/>
+      <parent link="quad_link"/>
+      <child link="quad${instance}_link"/>
     </joint>
-    <link name="${prefix}_link">
+    <link name="quad${instance}_link">
       <visual>
-        <geometry><cylinder length="${len}" radius="0.02"/></geometry>
-        <origin rpy="0 0 0" xyz="0 0 0"/>
+        <geometry><box size="0.01 0.1 0.03"/></geometry>
         <material name="red">
           <color rgba="${255/255} ${108/255} ${10/255} 1.0"/>
@@ -21,27 +18,23 @@
       <inertial>
         <origin rpy="0 0 0" xyz="0 0 0"/>
-        <mass value="${mass}"/>
-        <inertia ixx="${(len*len+len*len)*mass/12.0}" ixy="0.0" ixz="0.0"
-                 iyy="${(len*len+len*len)*mass/12.0}" iyz="0.0"
-                 izz="${(len*len+len*len)*mass/12.0}"/>
+        <mass value="0.05"/>
+        <inertia ixx="0.01" ixy="0.0" ixz="0.0"
+                    iyy="0.01" iyz="0.0"
+                        izz="0.01"/>
       </inertial>
-      <collision>
-        <origin rpy="0 0 0" xyz="0 0 0"/>
-        <geometry><cylinder length="${len}" radius="0.02"/></geometry>
-      </collision>
+      <collision><geometry><box size="0.01 0.1 0.03"/></geometry></collision>
     </link>
-    <joint name="${prefix}_optical_joint" type="fixed">
+    <!-- seems necessary to get a right side up image; see frameName below -->
+    <joint name="quad${instance}_optical_joint" type="fixed">
       <origin rpy="${-pi/2} 0 ${-pi/2}" xyz="0 0 0"/>
-      <parent link="${prefix}_link"/>
-      <child  link="${prefix}_optical_link"/>
+      <parent link="quad${instance}_link"/>
+      <child  link="quad${instance}_optical_link"/>
     </joint>
-    <!-- seems necessary to get a right side up image; see frameName below -->
-    <link name="${prefix}_optical_link" />
-    <!-- camera -->
-    <gazebo reference="${prefix}_link">
+    <link name="quad${instance}_optical_link" />
+    <gazebo reference="quad${instance}_link">
       <material>Gazebo/Black</material>
-      <sensor type="camera" name="${prefix}">
+      <sensor type="camera" name="quad${instance}">
         <update_rate>${fps}</update_rate>
-        <camera name="${prefix}">
+        <camera name="quad${instance}">
           <horizontal_fov>${fov}</horizontal_fov>
           <image>
@@ -52,5 +45,5 @@
           <clip>
             <near>0.02</near>
-            <far>3</far>
+            <far>30</far>
           </clip>
           <noise>
@@ -66,9 +59,8 @@
           <alwaysOn>true</alwaysOn>
           <updateRate>0.0</updateRate>
-          <cameraName>${prefix}</cameraName>
+          <cameraName>quad${instance}</cameraName>
           <imageTopicName>image_raw</imageTopicName>
           <cameraInfoTopicName>camera_info</cameraInfoTopicName>
-          <frameName>${prefix}_optical_link</frameName>
-          <hackBaseline>0.0</hackBaseline>
+          <frameName>quad${instance}_optical_link</frameName>
           <distortionK1>0.0</distortionK1>
           <distortionK2>0.0</distortionK2>
@@ -76,4 +68,5 @@
           <distortionT1>0.0</distortionT1>
           <distortionT2>0.0</distortionT2>
+          <robotNamespace>/</robotNamespace>
         </plugin>
       </sensor>

File: vehicle/vehicle_model/urdf/vehicle.xacro (robot description, xacro)
@@ -4,4 +4,5 @@
   <xacro:include filename="$(find vehicle_model)/urdf/wheel.xacro" />
   <xacro:include filename="$(find vehicle_model)/urdf/steering.xacro" />
+  <xacro:include filename="$(find camera_description)/urdf/quad_camera.xacro"/>
   <xacro:include filename="$(find camera_description)/urdf/monocular_camera.xacro"/>
   <xacro:include filename="$(find imu_description)/urdf/imu.xacro"/>
@@ -47,12 +48,12 @@
   <!-- ================ sensor to base_link xforms ================ -->
 	<xacro:property name="calibration" value="${load_yaml('$(find vehicle_model)/config/calibration.yaml')}"/>
-  <xacro:monocular_camera_macro suffix="cam_rl" parent="base_link" namespace="cam_rl"
-                                x="${calibration['base_link2camera']['x']}"
-                                y="${calibration['base_link2camera']['y']}"
-                                z="${calibration['base_link2camera']['z']}"
-                                roll="${calibration['base_link2camera']['roll']}"
-                                pitch="${calibration['base_link2camera']['pitch']}"
-                                yaw="${calibration['base_link2camera']['yaw']}"
-                                fps="6" width="1280" height="720" fov="1.6"/>
+  <xacro:quad_camera_macro prefix="up" parent="base_link"
+      x="${calibration['base_link2quad']['x']}"
+      y="${calibration['base_link2quad']['y']}"
+      z="${calibration['base_link2quad']['z']}"
+      roll="${calibration['base_link2quad']['roll']}"
+      pitch="${calibration['base_link2quad']['pitch']}"
+      yaw="${calibration['base_link2quad']['yaw']}"
+      fps="6" width="1280" height="720" fov="1.6"/>
   <xacro:imu_macro suffix="imu" parent="base_link" namespace=""
                    x="${calibration['base_link2imu']['x']}"

Commit message: Fix angle variance calculation

File: vehicle/sensor_model/camera/camera_description/urdf/D430IR.xacro (robot description, xacro)
@@ -18,8 +18,8 @@
       <inertial>
         <origin rpy="0 0 0" xyz="0 0 0"/>
-        <mass value="0.05"/>
-        <inertia ixx="0.01" ixy="0.0" ixz="0.0"
-                    iyy="0.01" iyz="0.0"
-                        izz="0.01"/>
+        <mass value="0.02"/>
+        <inertia ixx="0.0001" ixy="0.0" ixz="0.0"
+                    iyy="0.0001" iyz="0.0"
+                        izz="0.0001"/>
       </inertial>
       <collision><geometry><box size="0.01 0.1 0.03"/></geometry></collision>

File: vehicle/sensor_model/camera/camera_description/urdf/quad_camera.xacro (robot description, xacro)
@@ -23,7 +23,7 @@
         <origin rpy="0 0 0" xyz="0 0 0"/>
         <mass value="${mass}"/>
-        <inertia ixx="0.08" ixy="0.0" ixz="0.0"
-                    iyy="0.08" iyz="0.0"
-                        izz="0.01"/>
+        <inertia ixx="0.008" ixy="0.0" ixz="0.0"
+                    iyy="0.008" iyz="0.0"
+                        izz="0.001"/>
       </inertial>
       <collision>

File: vehicle/vehicle_model/urdf/vehicle.xacro (robot description, xacro)
@@ -22,5 +22,5 @@
   <xacro:property name="vehicle_width" value="${vehicle_info['vehicle_width']}"/>
   <xacro:property name="vehicle_height" value="${vehicle_info['vehicle_height']}"/>
-  <xacro:property name="vehicle_mass_height" value="0.5"/>
+  <xacro:property name="vehicle_mass_height" value="0.05"/>
   <!-- body-->
   <xacro:body_macro suffix="base"

Commit message: Estimate trailer pose with webcam

File: vehicle/sensor_model/camera/camera_description/urdf/D430IR.xacro (robot description, xacro)
@@ -12,5 +12,5 @@
       <visual>
         <geometry><box size="0.01 0.1 0.03"/></geometry>
-        <material name="red">
+        <material name="orange">
           <color rgba="${255/255} ${108/255} ${10/255} 1.0"/>
         </material>

File: vehicle/vehicle_model/urdf/vehicle.xacro (robot description, xacro)
@@ -55,6 +55,6 @@
       pitch="${calibration['base_link2quad']['pitch']}"
       yaw="${calibration['base_link2quad']['yaw']}"
-      fps="15" width="1280" height="720" fov="1.6"/>
-  <xacro:monocular_camera_macro prefix="up" parent="base_link"
+      fps="6" width="1280" height="720" fov="1.6"/>
+  <xacro:monocular_camera_macro prefix="webcam" parent="base_link"
       x="${calibration['base_link2camera']['x']}"
       y="${calibration['base_link2camera']['y']}"
@@ -63,4 +63,4 @@
       pitch="${calibration['base_link2camera']['pitch']}"
       yaw="${calibration['base_link2camera']['yaw']}"
-      fps="15" width="640" height="480" fov="2.0"/>
+      fps="15" width="640" height="480" fov="1.523"/> <!--H: 87.26 V: 64.96-->
 </robot>
