Commit message: Added rear_body and body_with_trailer xacro

File: vehicle/sensor_model/rear_bumper/rear_bumper_description/urdf/rear_bumper.xacro (robot description, xacro)
@@ -3,10 +3,10 @@
 <!-- <xacro:property name="pi" value="3.1415926835897931" /> -->
   <xacro:macro name="bumper_macro" params="parent">
-    <joint name="bumper_joint" type="fixed">
+    <joint name="rear_bumper_joint" type="fixed">
       <parent link="${parent}"/>
       <origin rpy="0 0 0" xyz="0.12 0 0.1"/>
-      <child  link="bumper_link"/>
+      <child  link="rear_bumper_link"/>
     </joint>
-    <link name="bumper_link">
+    <link name="rear_bumper_link">
       <!--pose>0.125 0 0.09  0 0 0</pose-->
       <inertial>
@@ -24,5 +24,5 @@
         </material>
       </visual>
-      <collision name="bumper_collision">
+      <collision name="rear_bumper_collision">
         <geometry>
           <box size="0.024 0.024 0.024"/>
@@ -30,17 +30,17 @@
       </collision>
    </link>
-    <gazebo reference="bumper_link">
+    <gazebo reference="rear_bumper_link">
      <material>Gazebo/Black</material>
-      <sensor name="bumper_sensor" type="contact"  >
+      <sensor name="rear_bumper_sensor" type="contact"  >
         <update_Rate>2</update_Rate>
         <always_on>true</always_on>
         <contact>
-          <collision>base_footprint_fixed_joint_lump__bumper_collision_collision_6</collision>
-          <topic>/contact_5wheel</topic>
+          <collision>base_footprint_fixed_joint_lump__rear_bumper_collision_collision_11</collision>
+          <topic>/rear_contact_5wheel</topic>
         </contact>
         <plugin name='bumper_sensor_plugin' filename='libgazebo_ros_bumper.so'>
           <alwaysOn>true</alwaysOn>
           <updateRate>2</updateRate>
-          <bumperTopicName>/contact_5wheel</bumperTopicName>
+          <bumperTopicName>/rear_contact_5wheel</bumperTopicName>
           <frameName>base_link</frameName>
         </plugin>
