Commit message: Bumper sensor still not working well

File: vehicle/sensor_model/bumper/bumper_description/urdf/bumper.xacro (robot description, xacro)
@@ -36,5 +36,5 @@
         <always_on>true</always_on>
         <contact>
-          <collision>base_footprint_fixed_joint_lump__bumper_collision_collision_7</collision>
+          <collision>base_footprint_fixed_joint_lump__bumper_collision_collision_6</collision>
           <topic>/contact_5wheel</topic>
         </contact>

Commit message: Tank turn

File: vehicle/sensor_model/bumper/bumper_description/urdf/bumper.xacro (robot description, xacro)
@@ -37,10 +37,10 @@
         <contact>
           <collision>base_footprint_fixed_joint_lump__bumper_collision_collision_6</collision>
-          <topic>/contact_5wheel</topic>
+          <topic>irrevant_contact_topic</topic>
         </contact>
         <plugin name='bumper_sensor_plugin' filename='libgazebo_ros_bumper.so'>
           <alwaysOn>true</alwaysOn>
           <updateRate>2</updateRate>
-          <bumperTopicName>/contact_5wheel</bumperTopicName>
+          <bumperTopicName>contact_5whl</bumperTopicName>
           <frameName>base_link</frameName>
         </plugin>

File: vehicle/vehicle_model/urdf/actuator.xacro (robot description, xacro)
@@ -41,3 +41,22 @@
     </actuator>
   </transmission>
+  <!-- rear wheel motor -->
+  <transmission name="wheel_left_rear_trans">
+    <type>transmission_interface/SimpleTransmission</type>
+    <joint name="wheel_left_rear_joint">
+      <hardwareInterface>hardware_interface/VelocityJointInterface</hardwareInterface>
+    </joint>
+    <actuator name="wheel_left_rear_motor">
+       <mechanismReduction>1</mechanismReduction>
+    </actuator>
+  </transmission>
+  <transmission name="wheel_right_rear_trans">
+    <type>transmission_interface/SimpleTransmission</type>
+    <joint name="wheel_right_rear_joint">
+      <hardwareInterface>hardware_interface/VelocityJointInterface</hardwareInterface>
+    </joint>
+    <actuator name="wheel_right_rear_motor">
+       <mechanismReduction>1</mechanismReduction>
+    </actuator>
+  </transmission>
 </robot>
